File: MCU - Power.kicad_sch (KiCad schematic)
At the start: 1 part

Commit message: Add 15v power system
Parts:
- added C1, C12, C16, C4: 100nF, Capacitor_SMD:C_0402_1005Metric, symbol JLCPCB_Basic_Capacitor_MLCC:100nF_0402_16V_X7R_±10%
- added C10, C14, C22, C23, C24, C3: 22uF, Capacitor_SMD:C_0805_2012Metric, symbol JLCPCB_Basic_Capacitor_MLCC:22uF_0805_25V_X5R_±20%
- added C11, C7: 4.7uF, Capacitor_SMD:C_0402_1005Metric, symbol JLCPCB_Basic_Capacitor_MLCC:4.7uF_0402_10V_X5R_±20%
- added C13, C5, C8: 1uF, Capacitor_SMD:C_0402_1005Metric, symbol JLCPCB_Basic_Capacitor_MLCC:1uF_0402_25V_X5R_±10%
- added C15: 22nF, Capacitor_SMD:C_0402_1005Metric, symbol JLCPCB_Basic_Capacitor_MLCC:22nF_0402_50V_X7R_±10%
- added C17: 6.8nF, Capacitor_SMD:C_0402_1005Metric, symbol JLCPCB_Basic_Capacitor_MLCC:6.8nF_0402_50V_X7R_±10%
- added C18, C20, C9: 10uF, Capacitor_SMD:C_0603_1608Metric, symbol JLCPCB_Basic_Capacitor_MLCC:10uF_0603_25V_X5R_±20%
- added C19, C25, C26, C27, C6: 470uF/35V, Capacitor_SMD:CP_Elec_8x10, symbol Device:C_Polarized
- added C2: 22uF, Capacitor_SMD:C_0603_1608Metric, symbol JLCPCB_Basic_Capacitor_MLCC:22uF_0603_6.3V_X5R_±20%
- added C21: 100nF, Capacitor_SMD:C_0402_1005Metric, symbol JLCPCB_Basic_Capacitor_MLCC:100nF_0402_50V_X7R_±10%
- added D1, D2: ES2J, Diode_SMD:D_SMA, symbol Device:D_Schottky
- added D3, D4, D5: BAT60B, Diode_SMD:D_SOD-323, symbol JLCPCB_Basic_Diode-Schottky:BAT60B
- added F1: 25A, symbol Device:Fuse
- added J1: USB_C_Receptacle_USB2.0_16P, Connector_USB:USB_C_Receptacle_HCTL_HC-TYPE-C-16P-01A, symbol Connector:USB_C_Receptacle_USB2.0_16P
- added J2, J3: Screw_Terminal_01x02, TerminalBlock_4Ucon:TerminalBlock_4Ucon_1x02_P3.50mm_Horizontal, symbol Connector:Screw_Terminal_01x02
- added J4: Conn_01x05, Connector_PinHeader_2.54mm:PinHeader_1x05_P2.54mm_Vertical, symbol Connector_Generic:Conn_01x05
- added J5: Conn_01x04, Connector_PinHeader_2.54mm:PinHeader_1x04_P2.54mm_Vertical, symbol Connector_Generic:Conn_01x04
- added J6: Screw_Terminal_01x02, symbol Connector:Screw_Terminal_01x02
- added L1, L2: 1.5uH, symbol Device:L
- added L3: 68uh/2A, Inductor_SMD:L_10.4x10.4_H4.8, symbol Device:L
- added Q1, Q2: AO3400A, Package_TO_SOT_SMD:SOT-23, symbol JLCPCB_Basic_Mosfet_NPN:AO3400A
- added Q5: AO3401A, Package_TO_SOT_SMD:SOT-23, symbol JLCPCB_Basic_Mosfet_PNP:AO3401A
- added R1, R10, R11, R12, R13, R2: 4.7k, Resistor_SMD:R_0402_1005Metric, symbol JLCPCB_Basic_Resistor:4.7kΩ_0402_±1%
- added R14: 6.8k, Resistor_SMD:R_0402_1005Metric, symbol JLCPCB_Basic_Resistor:6.8kΩ_0402_±1%
- added R15, R5, R6: 1k, Resistor_SMD:R_0402_1005Metric, symbol JLCPCB_Basic_Resistor:1kΩ_0402_±1%
- added R16, R19: R, symbol Device:R
- added R17, R18: 100k, Resistor_SMD:R_0402_1005Metric, symbol JLCPCB_Basic_Resistor:100kΩ_0402_±1%
- added R3, R4, R7, R8: 10k, Resistor_SMD:R_0402_1005Metric, symbol JLCPCB_Basic_Resistor:10kΩ_0402_±1%
- added R9: 1.2k, Resistor_SMD:R_0402_1005Metric, symbol JLCPCB_Basic_Resistor:1.2kΩ_0402_±1%
- added SW1, SW10, SW11, SW12, SW13, SW14, SW2, SW3, SW4, SW5, SW6, SW7, SW8, SW9: SW_Push, Button_Switch_SMD:SW_Push_1P1T_XKB_TS-1187A, symbol Switch:SW_Push
- added U2: TP4056-42-ESOP8, Package_SO:SOIC-8-1EP_3.9x4.9mm_P1.27mm_EP2.41x3.3mm_ThermalVias, symbol Battery_Management:TP4056-42-ESOP8
- added U3: XL1509-5.0, Package_SO:SOIC-8_3.9x4.9mm_P1.27mm, symbol Regulator_Switching:XL1509-5.0
- added U4: CH221K, Package_TO_SOT_SMD:SOT-23-6, symbol Interface_USB:CH221K
- added U5: TPS63031DSK, Package_SON:WSON-10-1EP_2.5x2.5mm_P0.5mm_EP1.2x2mm_ThermalVias, symbol Regulator_Switching:TPS63031DSK
- added U6: MP3429GL-Z, footprints:QFN-3x4_MP3429_MNP, symbol MP3429GL-Z:MP3429GL-Z
- gave numbers to parts that had none: 1
Connections:
- net GND: now reaches U1.1 (GND), U1.40 (GND), U1.41 (GND)
- net GND: now also C1.2, C10.2, C11.2, C12.2, C13.2, C14.2, C15.2, C18.2, C19.2, C2.2, C20.2, C21.2, C22.2, C23.2, C24.2, C25.2, C26.2, C27.2, C3.2, C4.2, C5.2, C6.2, C7.2, C8.2, C9.2, D5.2 (A), J1.A1 (GND), J1.A12 (GND), J1.B1 (GND), J1.B12 (GND), J1.SH (SHIELD), J4.1 (Pin_1), J5.1 (Pin_1), J6.2 (Pin_2), Q1.2 (S), Q2.2 (S), R1.2, R14.2, R18.2, R19.2, R2.2, R7.2, R8.2, R9.2, SW1.2, SW10.2, SW11.2, SW12.2, SW13.2, SW14.2, SW2.2, SW3.2, SW4.2, SW5.2, SW6.2, SW7.2, SW8.2, SW9.2, U2.1 (TEMP), U2.3 (GND), U2.9 (EPAD), U3.4 (~{EN}), U3.5 (GND), U3.6 (GND), U3.7 (GND), U3.8 (GND), U4.2 (GND), U5.11 (PGND), U5.3 (PGND), U5.9 (GND), U6.6 (AGND), U6.7 (PGND), U6.9 (FTY)
- net Solenoid: now reaches U1.10 (IO17)
- net Solenoid: now also R5.1
- net SDA - OLED: now reaches U1.11 (IO18)
- net SDA - OLED: now also J4.3 (Pin_3), R11.2
- net SCL - CAM: now reaches U1.12 (IO8)
- net SCL - CAM: now also J5.3 (Pin_3), R12.2
- net USB_D-: now reaches U1.13 (USB_D-)
- net USB_D-: now also J1.A7 (D-), J1.B7 (D-)
- net USB_D+: now reaches U1.14 (USB_D+)
- net USB_D+: now also J1.A6 (D+), J1.B6 (D+)
- net CAM - Clock: now reaches U1.15 (IO3)
- net CAM - Clock: now also J4.2 (Pin_2)
- net Button Pedal 2: now reaches U1.16 (IO46)
- net Button Pedal 2: now also SW13.1
- net SDA - CAM: now reaches U1.17 (IO9)
- net SDA - CAM: now also J5.2 (Pin_2), R13.2
- net Button A: now reaches U1.18 (IO10)
- net Button A: now also SW3.1
- net Button B: now reaches U1.19 (IO11)
- net Button B: now also SW4.1
- net +3.3V: now reaches U1.2 (3V3)
- net +3.3V: now also C1.1, C18.1, C2.1, C20.1, J4.5 (Pin_5), J5.4 (Pin_4), R10.1, R11.1, R12.1, R13.1, R3.1, R4.1, U5.1 (VOUT), U5.10 (FB)
- net Button C: now reaches U1.23 (IO21)
- net Button C: now also SW5.1
- net Button Pedal 1: now reaches U1.24 (IO47)
- net Button Pedal 1: now also SW14.1
- net Button Pump: now reaches U1.26 (IO45)
- net Button Pump: now also SW2.1
- net Button Home: now reaches U1.27 (IO0)
- net Button Home: now also SW6.1
- net EN: now reaches U1.3 (EN)
- net EN: now also R3.2
- net Button Select: now reaches U1.31 (IO38)
- net Button Select: now also SW7.1
- net Button Start: now reaches U1.32 (IO39)
- net Button Start: now also SW8.1
- net Button Up: now reaches U1.33 (IO40)
- net Button Up: now also SW9.1
- net Button Down: now reaches U1.34 (IO41)
- net Button Down: now also SW10.1
- net Button Left: now reaches U1.35 (IO42)
- net Button Left: now also SW11.1
- net Button Right: now reaches U1.38 (IO2)
- net Button Right: now also SW12.1
- net Button Trigger: now reaches U1.39 (IO1)
- net Button Trigger: now also SW1.1
- net SCL - OLED: now reaches U1.8 (IO15)
- net SCL - OLED: now also J4.4 (Pin_4), R10.2
- net Rumble: now reaches U1.9 (IO16)
- net Rumble: now also R6.1
- new net: Q1.1 (G), R5.2, R7.1
- new net: Q2.1 (G), R6.2, R8.1
- new net: D1.2 (A), J3.2 (Pin_2), Q2.3 (D)
- new net: C16.1, L2.2, U6.1 (SW)
- new net: C16.2, U6.13 (BST)
- new net: C11.1, U6.2 (VDD)
- new net: C15.1, U6.3 (SS)
- new net: C17.2, U6.4 (COMP)
- new net: R16.2, R19.1, U6.5 (FB)
- new net: C17.1, R14.1
- new net: D2.2 (A), J2.2 (Pin_2), Q1.3 (D)
- new net: R15.2, R17.1, U4.1 (VDD)
- new net: R17.2, U4.6 (CFG)
- new net: R9.1, U2.2 (PROG)
- new net: C12.1, U5.6 (EN), U5.7 (PS/SYNC), U5.8 (VINA)
- new net: D5.1 (K), L3.1, U3.2 (OUT)
- new net: F1.2, J6.1 (Pin_1)
- new net: L1.2, U5.2 (L2)
- new net: L1.1, U5.4 (L1)
- new net +15V: C21.1, C22.1, C23.1, C24.1, C25.1, C26.1, C27.1, D1.1 (K), D2.1 (K), D3.1 (K), J2.1 (Pin_1), J3.1 (Pin_1), R16.1, U6.8 (VOUT)
- new net +5V: C19.1, C4.1, D4.2 (A), L3.2, Q5.1 (G), R18.1, U2.4 (V_{CC}), U2.8 (CE), U3.3 (FB)
- new net +BATT: C10.1, C14.1, C3.1, C7.1, F1.1, L2.1, Q5.3 (D), U2.5 (BAT), U6.12 (VIN)
- new net BST_EN: U6.11 (EN)
- new net CC1: J1.A5 (CC1), R2.1, U4.4 (CC1)
- new net CC2: J1.B5 (CC2), R1.1, U4.5 (CC2)
- new net CHRG: U2.7 (~{CHRG})
- new net IO0: R4.2
- new net STDBY: U2.6 (~{STDBY})
- new net VBUS: C13.1, C5.1, C6.1, D3.2 (A), J1.A4 (VBUS), J1.A9 (VBUS), J1.B4 (VBUS), J1.B9 (VBUS), R15.1, U3.1 (VIN)
- new net VCC: C8.1, C9.1, D4.1 (K), Q5.2 (S), U5.5 (VIN)
- no-connect marks 0 -> 8
Other:
- note added: "https://blog.zakkemble.net/a-lithium-battery-charger-with-load-sharing/"
- note added: "https://ww1.microchip.com/downloads/en/AppNotes/01149c.pdf"
- moved on the sheet: U1
